Commit message: remove unused params, add typical params for keeping style, fix robot/macro and ros2_control plugin tag name because gazebo was not recognizing any ros2_control implementation

File: tm_description/xacro/macro.ros2_control.xacro (robot description, xacro)
@@ -1,6 +1,6 @@
 <?xml version="1.0"?>
 <robot xmlns:xacro="http://www.ros.org/wiki/xacro">
-    <xacro:macro name="tm5-700_ros2_control" params="name initial_positions_file">
-        <ros2_control name="${name}" type="system">
+    <xacro:macro name="tm5-700_ros2_control" params="ns prefix">
+        <ros2_control name="tm5-700_ros2_control" type="system">
             <hardware>
                 <plugin>gz_ros2_control/GazeboSimSystem</plugin>
